Commit message: Added real robot controllers and interfaces Added gazebo worlds Added octomap

File: streetbot4_description/urdf/jsnsr20y1.xacro (robot description, xacro)
@@ -14,14 +14,7 @@
             </inertial>
             <visual>
-                <origin xyz="0 -0.013 0" rpy="0 ${PI / 2} 0" />
+                <origin xyz="0 0 0" rpy="0 ${PI / 2} 0" />
                 <geometry>
-                    <cylinder radius="0.006" length="0.005"/>
-                </geometry>
-                <material name="Black" />
-            </visual>
-            <visual>
-                <origin xyz="0 0.013 0" rpy="0 ${PI / 2} 0" />
-                <geometry>
-                    <cylinder radius="0.006" length="0.005"/>
+                    <cylinder radius="0.010" length="0.005"/>
                 </geometry>
                 <material name="Black" />

File: streetbot4_description/urdf/streetbot4.xacro (robot description, xacro)
@@ -110,5 +110,5 @@
     </joint>
     <!-- Camera-->
-    <link name="camera_link">
+    <!-- <link name="camera_link">
         <inertial>
             <origin xyz="0 0 0" rpy="0 0 0" />
@@ -129,10 +129,12 @@
             </geometry>
         </collision>
-    </link>
-    <joint name="joint_sensor_camera" type="fixed">
-        <origin xyz="0.340 0 0.045" rpy="0 0 0"/>
+    </link> -->
+    <xacro:sensor_d435 name="camera" topics_ns="camera" parent="body_link" publish_pointcloud="true">
+        <origin xyz="0.330 0 0.035" rpy="0 0 0"/>
+    </xacro:sensor_d435>
+    <!-- <joint name="joint_sensor_camera" type="fixed">
         <parent link="body_link"/>
         <child link="camera_link"/>
-    </joint>
+    </joint> -->
     <!-- 4 Ultrasonic distance sensors -->
     <xacro:jsnsr20y1 parent="body_link" name="ultrasonic1">
