Commit message: Calculate component sizes and origin automatically from parameters

File: streetbot4_description/urdf/streetbot4.xacro (robot description, xacro)
@@ -12,4 +12,6 @@
     <xacro:property name="wheel_distance" value="0.249"/>
     <xacro:property name="wheel_width" value="0.086"/>
+    <xacro:property name="wheel_marker_length" value="0.03"/>
+    <xacro:property name="wheel_marker_width" value="0.005"/>
     <xacro:property name="mass" value="0.1"/>
     <xacro:property name="wheel_mass" value="0.2"/>
@@ -102,5 +104,5 @@
             <origin xyz="0 0 0" rpy="0 0 0" />
             <geometry>
-                <box size="0.03 0.005 0.005" />
+                <box size="${wheel_marker_length} ${wheel_marker_width} ${wheel_marker_width}" />
             </geometry>
             <material name="White" />
@@ -134,5 +136,5 @@
             <origin xyz="0 0 0" rpy="0 0 0" />
             <geometry>
-                <box size="0.03 0.005 0.005" />
+                <box size="${wheel_marker_length} ${wheel_marker_width} ${wheel_marker_width}" />
             </geometry>
             <material name="White" />
@@ -166,5 +168,5 @@
             <origin xyz="0 0 0" rpy="0 0 0" />
             <geometry>
-                <box size="0.03 0.005 0.005" />
+                <box size="${wheel_marker_length} ${wheel_marker_width} ${wheel_marker_width}" />
             </geometry>
             <material name="White" />
@@ -198,5 +200,5 @@
             <origin xyz="0 0 0" rpy="0 0 0" />
             <geometry>
-                <box size="0.03 0.005 0.005" />
+                <box size="${wheel_marker_length} ${wheel_marker_width} ${wheel_marker_width}" />
             </geometry>
             <material name="White" />
@@ -242,20 +244,20 @@
         <parent link="rear_left_wheel" />
         <child link="rear_left_wheel_marker" />
-        <origin xyz="0.015 0.0175 0" rpy="0 0 0" />
+        <origin xyz="${wheel_radius - wheel_marker_length / 2} ${wheel_width / 2 + wheel_marker_width / 2} 0" rpy="0 0 0" />
     </joint>
     <joint name="rear_right_wheel_to_marker" type="fixed">
         <parent link="rear_right_wheel" />
         <child link="rear_right_wheel_marker" />
-        <origin xyz="0.015 -0.0175 0" rpy="0 0 0" />
+        <origin xyz="${wheel_radius - wheel_marker_length / 2} -${wheel_width / 2 + wheel_marker_width / 2} 0" rpy="0 0 0" />
     </joint>
     <joint name="front_left_wheel_to_marker" type="fixed">
         <parent link="front_left_wheel" />
         <child link="front_left_wheel_marker" />
-        <origin xyz="0.015 0.0175 0" rpy="0 0 0" />
+        <origin xyz="${wheel_radius - wheel_marker_length / 2} ${wheel_width / 2 + wheel_marker_width / 2} 0" rpy="0 0 0" />
     </joint>
     <joint name="front_right_wheel_to_marker" type="fixed">
         <parent link="front_right_wheel" />
         <child link="front_right_wheel_marker" />
-        <origin xyz="0.015 -0.0175 0" rpy="0 0 0" />
+        <origin xyz="${wheel_radius - wheel_marker_length / 2} -${wheel_width / 2 + wheel_marker_width / 2} 0" rpy="0 0 0" />
     </joint>
 </robot>

Commit message: Fix robot model

File: streetbot4_description/urdf/streetbot4.xacro (robot description, xacro)
@@ -37,7 +37,7 @@
 		</visual>
 		<collision>
-			<origin xyz="0 0 ${clearance}" rpy="0 0 0" />
-            <geometry>
-                <box size="${wheel_distance + wheel_distance} ${wheel_separation - 0.04} ${body_height}"/>
+			<origin xyz="0 0 -0.015" rpy="${PI/2} 0 ${PI/2}" />
+            <geometry>
+                <mesh filename="package://streetbot4_description/meshes/streetbot4_body.stl" scale="0.001 0.001 0.001" />
             </geometry>
 		</collision>
@@ -62,5 +62,5 @@
         </inertial>
         <visual>
-            <origin xyz="0 0 -0.020" rpy="0 0 0" />
+            <origin xyz="0 0 0" rpy="0 0 0" />
             <geometry>
                 <cylinder radius="0.035" length="0.039"/>
@@ -76,5 +76,5 @@
     </link>
     <joint name="joint_sensor_laser" type="fixed">
-        <origin xyz="0 0 0.140" rpy="0 0 ${PI}"/>
+        <origin xyz="0 0 0.120" rpy="0 0 ${PI}"/>
         <parent link="body_link"/>
         <child link="rplidar_link"/>

Commit message: Added GPS, camera and ultrasonic sensor

File: streetbot4_description/urdf/streetbot4.xacro (robot description, xacro)
@@ -4,4 +4,7 @@
 	<!-- Matherials -->
 	<xacro:include filename="$(find streetbot4_description)/urdf/streetbot4_materials.xacro" />
+    <!-- Components -->
+    <xacro:include filename="$(find streetbot4_description)/urdf/jsnsr20y1.xacro" />
+    <xacro:include filename="$(find streetbot4_description)/urdf/jsnsr20y1.gazebo" />
     <!-- Gazebo parameters -->
     <xacro:include filename="$(find streetbot4_description)/urdf/streetbot4.gazebo" />
@@ -80,4 +83,69 @@
         <child link="rplidar_link"/>
     </joint>
+    <!-- GPS-->
+    <link name="gps_link">
+        <inertial>
+            <origin xyz="0 0 0" rpy="0 0 0" />
+            <mass value="0.1" />
+            <inertia ixx="0.0" ixy="0.0" ixz="0.0" iyy="0.0" iyz="0.0" izz="0.0" />
+        </inertial>
+        <visual>
+            <origin xyz="0 0 0" rpy="0 0 0" />
+            <geometry>
+                <box size="0.040 0.040 0.015" />
+            </geometry>
+            <material name="Green" />
+        </visual>
+        <collision>
+            <origin xyz="0 0 0" rpy="0 0 0"/>
+            <geometry>
+                <box size="0.040 0.040 0.015" />
+            </geometry>
+        </collision>
+    </link>
+    <joint name="joint_sensor_gps" type="fixed">
+        <origin xyz="0.200 0 0.105" rpy="0 0 0"/>
+        <parent link="body_link"/>
+        <child link="gps_link"/>
+    </joint>
+    <!-- Camera-->
+    <link name="camera_link">
+        <inertial>
+            <origin xyz="0 0 0" rpy="0 0 0" />
+            <mass value="0.1" />
+            <inertia ixx="0.0" ixy="0.0" ixz="0.0" iyy="0.0" iyz="0.0" izz="0.0" />
+        </inertial>
+        <visual>
+            <origin xyz="0 0 0" rpy="0 0 0" />
+            <geometry>
+                <box size="0.010 0.010 0.010" />
+            </geometry>
+            <material name="Green" />
+        </visual>
+        <collision>
+            <origin xyz="0 0 0" rpy="0 0 0"/>
+            <geometry>
+                <box size="0.010 0.010 0.010" />
+            </geometry>
+        </collision>
+    </link>
+    <joint name="joint_sensor_camera" type="fixed">
+        <origin xyz="0.340 0 0.045" rpy="0 0 0"/>
+        <parent link="body_link"/>
+        <child link="camera_link"/>
+    </joint>
+    <!-- 4 Ultrasonic distance sensors -->
+    <xacro:jsnsr20y1 parent="body_link" name="ultrasonic1">
+        <origin xyz="0.325 0.090 0.005" rpy="0 0.296705973 0"/>
+    </xacro:jsnsr20y1>
+    <xacro:jsnsr20y1 parent="body_link" name="ultrasonic2">
+        <origin xyz="0.325 -0.090 0.005" rpy="0 0.296705973 0"/>
+    </xacro:jsnsr20y1>
+    <xacro:jsnsr20y1 parent="body_link" name="ultrasonic3">
+        <origin xyz="-0.338 0.090 0.045" rpy="0 0.296705973 ${PI}"/>
+    </xacro:jsnsr20y1>
+    <xacro:jsnsr20y1 parent="body_link" name="ultrasonic4">
+        <origin xyz="-0.338 -0.090 0.045" rpy="0 0.296705973 ${PI}"/>
+    </xacro:jsnsr20y1>
     <!-- Wheels -->
     <link name="rear_left_wheel">

File: streetbot4_description/urdf/streetbot4_materials.xacro (robot description, xacro)
@@ -14,4 +14,7 @@
 		<color rgba="1.0 1.0 1.0 1.0"/>
 	</material>
+	<material name="Black">
+		<color rgba="0.0 0.0 0.0 1.0"/>
+	</material>
 	<material name="Yellow">
 		<color rgba="1.0 1.0 0.0 1.0"/>

Commit message: Fix description for on robot launch

File: streetbot4_description/urdf/streetbot4.xacro (robot description, xacro)
@@ -12,5 +12,5 @@
     <xacro:property name="body_height" value="0.17" />
     <xacro:property name="wheel_radius" value="0.108"/>
-    <xacro:property name="wheel_separation" value="0.344"/>
+    <xacro:property name="wheel_separation" value="0.47"/>
     <xacro:property name="wheel_distance" value="0.249"/>
     <xacro:property name="wheel_width" value="0.086"/>
@@ -110,5 +110,5 @@
     </joint>
     <!-- Camera-->
-    <!-- <link name="camera_link">
+    <link name="camera_link">
         <inertial>
             <origin xyz="0 0 0" rpy="0 0 0" />
@@ -129,12 +129,13 @@
             </geometry>
         </collision>
-    </link> -->
-    <xacro:sensor_d435 name="camera" topics_ns="camera" parent="body_link" publish_pointcloud="true">
+    </link>
+    <!--    <xacro:sensor_d435 name="camera" topics_ns="camera" parent="body_link" publish_pointcloud="true">
         <origin xyz="0.330 0 0.035" rpy="0 0 0"/>
-    </xacro:sensor_d435>
-    <!-- <joint name="joint_sensor_camera" type="fixed">
+    </xacro:sensor_d435> -->
+    <joint name="joint_sensor_camera" type="fixed">
         <parent link="body_link"/>
         <child link="camera_link"/>
-    </joint> -->
+        <origin xyz="0.330 0 0.035" rpy="0 0 0"/>
+    </joint>
     <!-- 4 Ultrasonic distance sensors -->
     <xacro:jsnsr20y1 parent="body_link" name="ultrasonic1">
